Commit message: chore(nav2): humble 기본 nav2_params.yaml로 교체 (jazzy 백업) + conflict 해결

File: linorobot2_description/urdf/2wd_properties.urdf.xacro (robot description, xacro)
@@ -1,22 +1,28 @@
 <?xml version="1.0"?>
 <robot xmlns:xacro="http://ros.org/wiki/xacro">
-  <xacro:property name="base_length" value="0.24" />
-  <xacro:property name="base_width" value="0.275" />
-  <xacro:property name="base_height" value="0.003" />
-  <xacro:property name="base_mass" value="1" />
-  <xacro:property name="wheel_radius" value="0.045" />
-  <xacro:property name="wheel_width" value="0.01" />
-  <xacro:property name="wheel_pos_x" value="0.0" />
-  <xacro:property name="wheel_pos_y" value="0.13" />
-  <xacro:property name="wheel_pos_z" value="-0.03" />
-  <xacro:property name="wheel_mass" value=".1" />
+  <xacro:property name="base_length" value="0.32" />
+  <xacro:property name="base_width" value="0.38" />
+  <xacro:property name="base_height" value="0.09" />
+  <xacro:property name="base_mass" value="13" />
+  <xacro:property name="base_mesh_file" value="" />
+  <xacro:property name="wheel_radius" value="0.0535" />
+  <xacro:property name="wheel_width" value="0.053" />
+  <!-- 앞 캐스터 1개 구성: 구동 바퀴를 중심보다 5cm 뒤로 배치해 후방 안정성 확보 -->
+  <xacro:property name="wheel_pos_x" value="-0.05" />
+  <!-- wheel_pos_y = base_width / 2 = 0.38 / 2 -->
+  <xacro:property name="wheel_pos_y" value="0.19" />
+  <!-- wheel_pos_z = -(base_height / 2) = -(0.09 / 2), 바퀴 중심을 본체 바닥면에 정렬 -->
+  <xacro:property name="wheel_pos_z" value="-0.045" />
+  <xacro:property name="wheel_mass" value="0.3" />
   <xacro:property name="wheel_torque" value="20" />
   <xacro:property name="front_caster_wheel" value="true" />
-  <xacro:property name="rear_caster_wheel" value="true" />
+  <xacro:property name="rear_caster_wheel" value="false" />
+  <xacro:property name="wheel_mesh_file" value="" />
   <xacro:property name="laser_pose">
-    <origin xyz="0.12 0 0.33" rpy="0 0 0"/>
+    <origin xyz="0.0 0 0.095" rpy="0 0 0"/>
   </xacro:property>
+  <!-- 깊이 카메라: 본체 전면 중앙 높이 -->
   <xacro:property name="depth_sensor_pose">
-    <origin xyz="0.14 0.0 0.045" rpy="0 0 0"/>
+    <origin xyz="0.16 0.0 0.5" rpy="0 0 0"/>
   </xacro:property>
   <xacro:property name="rear_camera_sensor_pose">

File: linorobot2_description/urdf/sensors/depth_sensor.urdf.xacro (robot description, xacro)
@@ -1,58 +1,49 @@
 <robot xmlns:xacro="http://ros.org/wiki/xacro">
-  <xacro:property name="M_PI" value="3.1415926535897931" />
   <xacro:macro name="depth_sensor" params="*origin">
+    <!-- Intel RealSense L515 -->
     <link name="camera_link">
       <visual>
         <origin xyz="0 0 0" rpy="0 0 0"/>
         <geometry>
-          <box size="0.030 0.124 0.030"/>
-          <!-- <mesh filename="" scale="0.001 0.001 0.001"/> -->
+          <mesh filename="file:///opt/ros/humble/share/realsense2_description/meshes/l515.dae"/>
         </geometry>
-        <material name="red">
-          <color rgba="0.416 0.051 0.047 1.0"/>
-        </material>
       </visual>
       <collision>
-        <origin xyz="0 0 0" rpy="0 0 0"/>
+        <!-- L515: 직경 61mm, 두께 26mm 원통으로 근사 -->
+        <origin xyz="0 0 0" rpy="0 1.5708 0"/>
         <geometry>
-          <box size="0.030 0.124 0.030"/>
+          <cylinder radius="0.0305" length="0.026"/>
         </geometry>
       </collision>
       <inertial>
         <origin xyz="0 0 0" rpy="0 0 0"/>
-        <mass value="0.135"/>
-        <inertia ixx="${(1/12) * 0.135 * ((0.124  * 0.124)  + (0.030 * 0.030))}" ixy="0.0" ixz="0.0"
-                 iyy="${(1/12) * 0.135 * ((0.030 * 0.030) + (0.030 * 0.030))}" iyz="0.0"
-                 izz="${(1/12) * 0.135 * ((0.030 * 0.030) + (0.124  * 0.124))}"/>
+        <mass value="0.1"/>
+        <inertia ixx="0.000025" ixy="0.0" ixz="0.0"
+                 iyy="0.000025" iyz="0.0"
+                 izz="0.000025"/>
       </inertial>
     </link>
-    <gazebo reference="camera_link">
-      <visual>
-        <material>
-          <ambient>0.416 0.051 0.047 1.0</ambient>
-          <diffuse>0.416 0.051 0.047 1.0</diffuse>
-          <specular>0.416 0.051 0.047 1.0</specular>
-          <emissive>0.416 0.051 0.047 1.0</emissive>
-        </material>
-      </visual>
-    </gazebo>rgb(213,28,40)
     <joint name="camera_to_base_link" type="fixed">
       <parent link="base_link"/>
       <child link="camera_link"/>
-      <xacro:insert_block name="origin" />
+      <xacro:insert_block name="origin"/>
     </joint>
     <link name="camera_depth_link"/>
     <joint name="camera_depth_joint" type="fixed">
-      <origin xyz="0 0 0" rpy="-1.57 0 -1.57"/>
+      <origin xyz="0 0 0" rpy="-1.5708 0 -1.5708"/>
       <parent link="camera_link"/>
       <child link="camera_depth_link"/>
     </joint>
-    <!-- https://github.com/ros-simulation/gazebo_ros_pkgs/wiki/ROS-2-Migration:-Camera#gazebo_ros_camera -->
+    <!-- Gazebo Harmonic rgbd_camera — L515 스펙 -->
     <gazebo reference="camera_link">
-      <sensor name="camera" type="depth">
+      <sensor name="camera" type="rgbd_camera">
+        <topic>camera</topic>
+        <update_rate>10.0</update_rate>
         <always_on>true</always_on>
-        <update_rate>30.0</update_rate>
-        <camera name="camera">
-          <horizontal_fov>1.50098</horizontal_fov>
+        <visualize>true</visualize>
+        <camera>
+          <optical_frame_id>camera_depth_link</optical_frame_id>
+          <!-- L515 depth FOV: 70° horizontal = 1.2217 rad -->
+          <horizontal_fov>1.2217</horizontal_fov>
           <image>
             <width>640</width>
@@ -60,4 +51,9 @@
             <format>R8G8B8</format>
           </image>
+          <clip>
+            <!-- L515 depth range: 0.25m ~ 9.0m -->
+            <near>0.25</near>
+            <far>9.0</far>
+          </clip>
         </camera>
         <plugin name="depth_camera_controller" filename="libgazebo_ros_camera.so">

Commit message: feat: AED 시연 환경 통합 변경 (2026-05-12)
- STVL(spatio_temporal_voxel_layer) 도입: VoxelLayer/ObstacleLayer → STVL, L515 PC2 직접 입력
- pointcloud_to_laserscan 노드 제거, scan_layers.yaml 삭제
- URDF: base box CAD 실측 (0.470x0.400x0.490m), 라이다 충돌 회피, 메쉬 file://$(find) 경로
- mapping/navigation 모드 분리: mapping.launch.py 신규, slam.launch.py 삭제
- navigation.launch.py 리팩터링 (map_server + AMCL + Nav2, SLAM 꺼짐)
- AMCL set_initial_pose 자동화
- footprint 캐스터 영역 포함, velocity_smoother CLOSED_LOOP, min_y_velocity 정상화
- bringup.launch.py 정리 (vesc_bridge 제거, description.launch.py 호출 추가)
- gazebo.launch.py 기본 world aed_corridor, --verbose 제거, env 검증 추가
- description.rviz 4WD → 2WD 갱신, scan_low/high 시각화 제거
- navigate_w_obstacle_wait.xml 주석을 실제 동작과 일치
- navigation.yaml Jazzy 잔재 경고 주석

File: linorobot2_description/urdf/2wd_properties.urdf.xacro (robot description, xacro)
@@ -1,17 +1,25 @@
 <?xml version="1.0"?>
 <robot xmlns:xacro="http://ros.org/wiki/xacro">
-  <xacro:property name="base_length" value="0.32" />
-  <xacro:property name="base_width" value="0.38" />
-  <xacro:property name="base_height" value="0.09" />
+  <!-- 충돌 박스: 본체 평판만 (라이다 마운트 제외)
+       Visual STL은 전체 형상 유지하지만, 충돌 박스가 라이다 위치를 포함하면
+       Gazebo lidar ray가 박스 내벽을 hit하여 phantom obstacle 발생 → 박스 상단을 라이다 아래로 -->
+  <xacro:property name="base_length" value="0.470" />
+  <xacro:property name="base_width" value="0.400" />
+  <xacro:property name="base_height" value="0.490" />
+  <!-- Z 범위: -0.102 ~ 0.388 (라이다 0.420 아래 3.2cm 마진) -->
+  <xacro:property name="base_origin_x" value="0.115" />
+  <xacro:property name="base_origin_y" value="0.000" />
+  <xacro:property name="base_origin_z" value="0.143" />
   <xacro:property name="base_mass" value="13" />
-  <xacro:property name="base_mesh_file" value="" />
-  <xacro:property name="wheel_radius" value="0.0535" />
-  <xacro:property name="wheel_width" value="0.053" />
+  <xacro:property name="base_mesh_file" value="file://$(find linorobot2_description)/meshes/aed_robot.stl" />
+  <!-- CAD 실측: 인휠 직경 139mm → 반지름 69.5mm -->
+  <xacro:property name="wheel_radius" value="0.0695" />
+  <xacro:property name="wheel_width" value="0.0385" />
   <!-- 앞 캐스터 1개 구성: 구동 바퀴를 중심보다 5cm 뒤로 배치해 후방 안정성 확보 -->
   <xacro:property name="wheel_pos_x" value="-0.05" />
-  <!-- wheel_pos_y = base_width / 2 = 0.38 / 2 -->
-  <xacro:property name="wheel_pos_y" value="0.19" />
-  <!-- wheel_pos_z = -(base_height / 2) = -(0.09 / 2), 바퀴 중심을 본체 바닥면에 정렬 -->
-  <xacro:property name="wheel_pos_z" value="-0.045" />
+  <!-- CAD 실측: 트랙폭 340mm / 2 = 170mm -->
+  <xacro:property name="wheel_pos_y" value="0.17" />
+  <!-- 바퀴 중심: base_link 기준 z=-0.09m (인휠모터 축 높이, 본체 밑판 57.5mm 위에 본체가 있도록) -->
+  <xacro:property name="wheel_pos_z" value="-0.09" />
   <xacro:property name="wheel_mass" value="0.3" />
   <xacro:property name="wheel_torque" value="20" />
@@ -19,10 +27,11 @@
   <xacro:property name="rear_caster_wheel" value="false" />
   <xacro:property name="wheel_mesh_file" value="" />
+  <!-- CAD 실측: RPLIDAR [87] 상단(스캔면) STEP Z=417mm -->
   <xacro:property name="laser_pose">
-    <origin xyz="0.0 0 0.095" rpy="0 0 0"/>
+    <origin xyz="0.08 0.0 0.420" rpy="0 0 0"/>
   </xacro:property>
-  <!-- 깊이 카메라: 본체 전면 중앙 높이 -->
+  <!-- CAD 실측: camera_module [40] STEP(51,-8,358)mm -->
   <xacro:property name="depth_sensor_pose">
-    <origin xyz="0.16 0.0 0.5" rpy="0 0 0"/>
+    <origin xyz="0.243 0.0 0.361" rpy="0 0 0"/>
   </xacro:property>
   <xacro:property name="rear_camera_sensor_pose">

File: linorobot2_description/urdf/mech/base.urdf.xacro (robot description, xacro)
@@ -1,19 +1,27 @@
 <?xml version="1.0"?>
 <robot xmlns:xacro="http://ros.org/wiki/xacro">
-  <xacro:macro name="base" params="length width height mass wheel_radius wheel_pos_z">
+  <xacro:macro name="base" params="length width height mass wheel_radius wheel_pos_z origin_x origin_y origin_z">
     <link name="base_footprint"/>
     <link name="base_link">
       <visual>
-        <origin xyz="0 0 0" rpy="0 0 0"/>
+        <origin xyz="0.235 -0.050 0.003" rpy="0 0 1.5708"/>
         <geometry>
-          <box size="${length} ${width} ${height}"/>
-          <!-- <mesh filename="" scale="0.001 0.001 0.001"/> -->
+          <mesh filename="${base_mesh_file}" scale="0.001 0.001 0.001"/>
         </geometry>
-        <material name="yellow">
-          <color rgba="0.8784 0.6627 0.6627 1.0"/>
+        <material name="robot_body">
+          <color rgba="0.3 0.3 0.3 1.0"/>
         </material>
       </visual>
+    <gazebo reference="base_link">
+      <visual>
+        <material>
+          <ambient>0.3 0.3 0.3 1.0</ambient>
+          <diffuse>0.5 0.5 0.5 1.0</diffuse>
+          <specular>0.2 0.2 0.2 1.0</specular>
+        </material>
+      </visual>
+    </gazebo>
       <collision>
-        <origin xyz="0 0 0" rpy="0 0 0"/>
+        <origin xyz="${origin_x} ${origin_y} ${origin_z}" rpy="0 0 0"/>
         <geometry>
           <box size="${length} ${width} ${height}"/>
@@ -21,5 +29,5 @@
       </collision>
       <inertial>
-        <origin xyz="0 0 0" rpy="0 0 0"/>
+        <origin xyz="${origin_x} ${origin_y} ${origin_z}" rpy="0 0 0"/>
         <mass value="${mass}"/>
         <inertia ixx="${(1/12) * mass * ((width  * width)  + (height * height))}" ixy="0.0" ixz="0.0"
@@ -28,14 +36,4 @@
       </inertial>
     </link>
-    <gazebo reference="base_link">
-      <visual>
-        <material>
-          <ambient>0.8392 0.6314 0.0 1.0</ambient>
-          <diffuse>0.8392 0.6314 0.0 1.0</diffuse>
-          <specular>0.99 0.99 0.99 1.0</specular>
-          <emissive>0.0 0.0 0.0 0.0</emissive>
-        </material>
-      </visual>
-    </gazebo>
     <joint name="base_to_footprint" type="fixed">
       <parent link="base_footprint"/>

File: linorobot2_description/urdf/mech/caster_wheel.urdf.xacro (robot description, xacro)
@@ -1,12 +1,7 @@
 <?xml version="1.0"?>
 <robot xmlns:xacro="http://ros.org/wiki/xacro">
-  <xacro:macro name="caster_wheel" params="side mass base_length wheel_radius wheel_pos_z">
-    <xacro:property name="caster_wheel_radius" value="${(wheel_radius - wheel_pos_z) / 2}" />
-    <xacro:if value="${side == 'front'}">
-        <xacro:property name="caster_wheel_x" value="${(base_length / 2) - caster_wheel_radius}" />
-    </xacro:if>
-    <xacro:if value="${side == 'rear'}">
-        <xacro:property name="caster_wheel_x" value="${-(base_length / 2) + caster_wheel_radius}" />
-    </xacro:if>
+  <xacro:macro name="caster_wheel" params="side mass caster_x caster_radius wheel_radius wheel_pos_z">
+    <xacro:property name="caster_wheel_radius" value="${caster_radius}" />
+    <xacro:property name="caster_wheel_x" value="${caster_x}" />
     <link name="${side}_caster_wheel_link">
       <visual>
@@ -40,5 +35,5 @@
       <parent link="base_link"/>
       <child link="${side}_caster_wheel_link"/>
-      <origin xyz="${caster_wheel_x} 0 -${caster_wheel_radius}" rpy="0 0 0"/>
+      <origin xyz="${caster_wheel_x} 0 -0.100" rpy="0 0 0"/>
     </joint>
   </xacro:macro>

File: linorobot2_description/urdf/robots/2wd.urdf.xacro (robot description, xacro)
@@ -17,4 +17,7 @@
     wheel_radius="${wheel_radius}"
     wheel_pos_z="${wheel_pos_z}"
+    origin_x="${base_origin_x}"
+    origin_y="${base_origin_y}"
+    origin_z="${base_origin_z}"
 />
   <xacro:wheel
@@ -40,5 +43,6 @@
       side="front"
       mass="0.01"
-      base_length="${base_length}"
+      caster_x="0.241"
+      caster_radius="0.060"
       wheel_radius="${wheel_radius}"
       wheel_pos_z="${wheel_pos_z}"
@@ -49,5 +53,6 @@
       side="rear"
       mass="0.01"
-      base_length="${base_length}"
+      caster_x="-0.241"
+      caster_radius="0.060"
       wheel_radius="${wheel_radius}"
       wheel_pos_z="${wheel_pos_z}"

File: linorobot2_description/urdf/sensors/depth_sensor.urdf.xacro (robot description, xacro)
@@ -35,13 +35,11 @@
       <child link="camera_depth_link"/>
     </joint>
-    <!-- Gazebo Harmonic rgbd_camera — L515 스펙 -->
+    <!-- Gazebo Classic 11 depth camera — L515 스펙 -->
     <gazebo reference="camera_link">
-      <sensor name="camera" type="rgbd_camera">
-        <topic>camera</topic>
+      <sensor name="camera" type="depth">
+        <always_on>true</always_on>
         <update_rate>10.0</update_rate>
-        <always_on>true</always_on>
-        <visualize>true</visualize>
-        <camera>
-          <optical_frame_id>camera_depth_link</optical_frame_id>
+        <visualize>false</visualize>
+        <camera name="camera">
           <!-- L515 depth FOV: 70° horizontal = 1.2217 rad -->
           <horizontal_fov>1.2217</horizontal_fov>
@@ -52,5 +50,4 @@
           </image>
           <clip>
-            <!-- L515 depth range: 0.25m ~ 9.0m -->
             <near>0.25</near>
             <far>9.0</far>
@@ -58,26 +55,8 @@
         </camera>
         <plugin name="depth_camera_controller" filename="libgazebo_ros_camera.so">
-          <ros>
-            <remapping>/camera/camera_info:=/camera/color/camera_info</remapping>
-            <remapping>/camera/image_raw:=/camera/color/image_raw</remapping>
-            <remapping>/camera/points:=/camera/depth/color/points</remapping>
-            <remapping>/camera/depth/image_raw:=/camera/depth/image_rect_raw</remapping>
-            <qos>
-              <topic name="/camera/depth/color/points">
-                <publisher>
-                  <reliability>best_effort</reliability>
-                </publisher>
-              </topic>
-            </qos>
-          </ros>
-          <min_depth>0.015</min_depth>
-          <max_depth>3.0</max_depth>
-          <hack_baseline>0.07</hack_baseline>
+          <camera_name>camera</camera_name>
           <frame_name>camera_depth_link</frame_name>
-          <distortion_k1>0.00000001</distortion_k1>
-          <distortion_k2>0.00000001</distortion_k2>
-          <distortion_k3>0.00000001</distortion_k3>
-          <distortion_t1>0.00000001</distortion_t1>
-          <distortion_t2>0.00000001</distortion_t2>
+          <min_depth>0.25</min_depth>
+          <max_depth>9.0</max_depth>
         </plugin>
       </sensor>

File: linorobot2_description/urdf/sensors/laser.urdf.xacro (robot description, xacro)
@@ -4,7 +4,7 @@
     <link name="${frame_id}">
       <visual>
-        <origin xyz="0 0 -0.025" rpy="0 0 0"/>
+        <origin xyz="0 0 -0.015" rpy="0 0 0"/>
         <geometry>
-          <cylinder radius="0.0375" length="0.05"/>
+          <cylinder radius="0.0375" length="0.030"/>
         </geometry>
         <material name="green">
@@ -13,7 +13,7 @@
       </visual>
       <collision>
-        <origin xyz="0 0 -0.025" rpy="0 0 0"/>
+        <origin xyz="0 0 -0.015" rpy="0 0 0"/>
         <geometry>
-          <cylinder radius="0.0375" length="0.05"/>
+          <cylinder radius="0.0375" length="0.030"/>
         </geometry>
       </collision>
