Commit message: fix: 실측 track_width 적용 (340mm → 294mm)
- URDF wheel_pos_y: 0.17 → 0.147
- Nav2 footprint y: ±0.19 → ±0.17 (안전 마진 포함)

Co-Authored-By: Claude Sonnet 4.6 <noreply@anthropic.com>

File: linorobot2_description/urdf/2wd_properties.urdf.xacro (robot description, xacro)
@@ -18,6 +18,6 @@
   <!-- 앞 캐스터 1개 구성: 구동 바퀴를 중심보다 5cm 뒤로 배치해 후방 안정성 확보 -->
   <xacro:property name="wheel_pos_x" value="-0.05" />
-  <!-- CAD 실측: 트랙폭 340mm / 2 = 170mm -->
-  <xacro:property name="wheel_pos_y" value="0.17" />
+  <!-- 실측: 트랙폭 294mm / 2 = 147mm (CAD 340mm → 실측 보정) -->
+  <xacro:property name="wheel_pos_y" value="0.147" />
   <!-- 바퀴 중심: base_link 기준 z=-0.09m (인휠모터 축 높이, 본체 밑판 57.5mm 위에 본체가 있도록) -->
   <xacro:property name="wheel_pos_z" value="-0.09" />

Commit message: fix: 실측 기반 footprint/base_box 보정
- footprint: 뒷면 -0.125 (회전축에서 75mm), 앞면 +0.345 (STL 470mm)
- base_origin_x: 0.115 → 0.110 (footprint 중심 일치)

Co-Authored-By: Claude Sonnet 4.6 <noreply@anthropic.com>

File: linorobot2_description/urdf/2wd_properties.urdf.xacro (robot description, xacro)
@@ -8,5 +8,5 @@
   <xacro:property name="base_height" value="0.490" />
   <!-- Z 범위: -0.102 ~ 0.388 (라이다 0.420 아래 3.2cm 마진) -->
-  <xacro:property name="base_origin_x" value="0.115" />
+  <xacro:property name="base_origin_x" value="0.110" />
   <xacro:property name="base_origin_y" value="0.000" />
   <xacro:property name="base_origin_z" value="0.143" />

Commit message: fix: 시뮬 카메라 방향 반전 (뒤→앞) rpy 3.14159→0
Co-Authored-By: Claude Sonnet 4.6 <noreply@anthropic.com>

File: linorobot2_description/urdf/2wd_properties.urdf.xacro (robot description, xacro)
@@ -36,5 +36,5 @@
   </xacro:property>
   <xacro:property name="rear_camera_sensor_pose">
-    <origin xyz="-0.14 0.0 0.045" rpy="0 0 3.14159"/>
+    <origin xyz="-0.14 0.0 0.045" rpy="0 0 0"/>
   </xacro:property>
 </robot>

Commit message: fix: 시뮬 RGB 카메라 위치를 L515 depth_sensor와 동일하게 (0.243, 0, 0.361)
기존 (-0.14, 0, 0.045)는 본체 내부였음

Co-Authored-By: Claude Sonnet 4.6 <noreply@anthropic.com>

File: linorobot2_description/urdf/2wd_properties.urdf.xacro (robot description, xacro)
@@ -35,6 +35,7 @@
     <origin xyz="0.243 0.0 0.361" rpy="0 0 0"/>
   </xacro:property>
+  <!-- 시뮬용 RGB 카메라: depth_sensor와 동일 위치 (L515 마운트) -->
   <xacro:property name="rear_camera_sensor_pose">
-    <origin xyz="-0.14 0.0 0.045" rpy="0 0 0"/>
+    <origin xyz="0.243 0.0 0.361" rpy="0 0 0"/>
   </xacro:property>
 </robot>

Commit message: fix: mesh 경로 file://\$(find) → package:// (크로스머신 RViz)
Jetson에서 \$(find)가 절대경로로 해석되어 노트북에서 STL 못 찾던 문제

Co-Authored-By: Claude Sonnet 4.6 <noreply@anthropic.com>

File: linorobot2_description/urdf/2wd_properties.urdf.xacro (robot description, xacro)
@@ -12,5 +12,5 @@
   <xacro:property name="base_origin_z" value="0.143" />
   <xacro:property name="base_mass" value="13" />
-  <xacro:property name="base_mesh_file" value="file://$(find linorobot2_description)/meshes/aed_robot.stl" />
+  <xacro:property name="base_mesh_file" value="package://linorobot2_description/meshes/aed_robot.stl" />
   <!-- CAD 실측: 인휠 직경 139mm → 반지름 69.5mm -->
   <xacro:property name="wheel_radius" value="0.0695" />

Commit message: fix(urdf): base_link를 회전중심으로 이동 + IMU/Optical Flow 좌표 입력
차분구동 odom_integrator는 base_link=회전중심(양 바퀴 축 중점)을
가정한다. 기존 base_link는 회전중심에서 +0.05m 앞에 있어 회전 시
odom이 ω×r만큼 횡방향으로 휘둘리는 문제 수정.

base_link 원점을 회전중심으로 이동, 영향받는 모든 좌표 +0.05 보정:
- wheel_pos_x 0.0, caster_x ±0.241→0.291/-0.191
- laser 0.13, depth_sensor/rear_camera 0.293
- base mesh visual 0.285, base_origin_x 0.160
- Nav2 footprint x: 앞면 0.395, 뒷면 -0.075

추가: IMU/Optical Flow URDF 좌표 실측 반영 (회전중심 기준)
- imu_link: xyz=-0.0075 0 0.0135, x축이 로봇 앞 방향과 일치(rpy=0)
- optical_flow_link 신규: xyz=0 0 -0.0955

Co-Authored-By: Claude Opus 4.7 (1M context) <noreply@anthropic.com>

File: linorobot2_description/urdf/2wd_properties.urdf.xacro (robot description, xacro)
@@ -8,5 +8,5 @@
   <xacro:property name="base_height" value="0.490" />
   <!-- Z 범위: -0.102 ~ 0.388 (라이다 0.420 아래 3.2cm 마진) -->
-  <xacro:property name="base_origin_x" value="0.110" />
+  <xacro:property name="base_origin_x" value="0.160" />
   <xacro:property name="base_origin_y" value="0.000" />
   <xacro:property name="base_origin_z" value="0.143" />
@@ -16,6 +16,6 @@
   <xacro:property name="wheel_radius" value="0.0695" />
   <xacro:property name="wheel_width" value="0.0385" />
-  <!-- 앞 캐스터 1개 구성: 구동 바퀴를 중심보다 5cm 뒤로 배치해 후방 안정성 확보 -->
-  <xacro:property name="wheel_pos_x" value="-0.05" />
+  <!-- base_link = 회전중심 (양 바퀴 축 중점). 바퀴는 base_link 원점에 위치 -->
+  <xacro:property name="wheel_pos_x" value="0.0" />
   <!-- 실측: 트랙폭 294mm / 2 = 147mm (CAD 340mm → 실측 보정) -->
   <xacro:property name="wheel_pos_y" value="0.147" />
@@ -29,13 +29,13 @@
   <!-- CAD 실측: RPLIDAR [87] 상단(스캔면) STEP Z=417mm -->
   <xacro:property name="laser_pose">
-    <origin xyz="0.08 0.0 0.420" rpy="0 0 0"/>
+    <origin xyz="0.13 0.0 0.420" rpy="0 0 0"/>
   </xacro:property>
   <!-- CAD 실측: camera_module [40] STEP(51,-8,358)mm -->
   <xacro:property name="depth_sensor_pose">
-    <origin xyz="0.243 0.0 0.361" rpy="0 0 0"/>
+    <origin xyz="0.293 0.0 0.361" rpy="0 0 0"/>
   </xacro:property>
   <!-- 시뮬용 RGB 카메라: depth_sensor와 동일 위치 (L515 마운트) -->
   <xacro:property name="rear_camera_sensor_pose">
-    <origin xyz="0.243 0.0 0.361" rpy="0 0 0"/>
+    <origin xyz="0.293 0.0 0.361" rpy="0 0 0"/>
   </xacro:property>
 </robot>

File: linorobot2_description/urdf/mech/base.urdf.xacro (robot description, xacro)
@@ -5,5 +5,5 @@
     <link name="base_link">
       <visual>
-        <origin xyz="0.235 -0.050 0.003" rpy="0 0 1.5708"/>
+        <origin xyz="0.285 -0.050 0.003" rpy="0 0 1.5708"/>
         <geometry>
           <mesh filename="${base_mesh_file}" scale="0.001 0.001 0.001"/>

File: linorobot2_description/urdf/robots/2wd.urdf.xacro (robot description, xacro)
@@ -6,4 +6,5 @@
   <xacro:include filename="$(find linorobot2_description)/urdf/mech/caster_wheel.urdf.xacro" />
   <xacro:include filename="$(find linorobot2_description)/urdf/sensors/imu.urdf.xacro" />
+  <xacro:include filename="$(find linorobot2_description)/urdf/sensors/optical_flow.urdf.xacro" />
   <xacro:include filename="$(find linorobot2_description)/urdf/sensors/generic_laser.urdf.xacro" />
   <xacro:include filename="$(find linorobot2_description)/urdf/sensors/depth_sensor.urdf.xacro" />
@@ -43,5 +44,5 @@
       side="front"
       mass="0.01"
-      caster_x="0.241"
+      caster_x="0.291"
       caster_radius="0.060"
       wheel_radius="${wheel_radius}"
@@ -53,5 +54,5 @@
       side="rear"
       mass="0.01"
-      caster_x="-0.241"
+      caster_x="-0.191"
       caster_radius="0.060"
       wheel_radius="${wheel_radius}"
@@ -60,4 +61,5 @@
   </xacro:if>
   <xacro:imu/>
+  <xacro:optical_flow/>
   <xacro:generic_laser>
     <xacro:insert_block name="laser_pose" />

File: linorobot2_description/urdf/sensors/imu.urdf.xacro (robot description, xacro)
@@ -5,5 +5,5 @@
       <parent link="base_link"/>
       <child link="imu_link"/>
-      <origin xyz="0 0 0" rpy="0 0 0"/>
+      <origin xyz="-0.0075 0 0.0135" rpy="0 0 0"/>
     </joint>
     <gazebo reference="imu_link">

Commit message: fix(urdf): laser frame yaw=pi (라이다 180° 회전 마운트 보정)
실측 결과 라이다가 180° 회전된 상태로 마운트됨. sllidar inverted: True와
조합하여 RViz상 장애물 방향이 실제와 일치하도록 frame yaw=pi 적용.

Co-Authored-By: Claude Opus 4.7 (1M context) <noreply@anthropic.com>

File: linorobot2_description/urdf/2wd_properties.urdf.xacro (robot description, xacro)
@@ -27,7 +27,8 @@
   <xacro:property name="rear_caster_wheel" value="false" />
   <xacro:property name="wheel_mesh_file" value="" />
-  <!-- CAD 실측: RPLIDAR [87] 상단(스캔면) STEP Z=417mm -->
+  <!-- CAD 실측: RPLIDAR [87] 상단(스캔면) STEP Z=417mm
+       rpy yaw=pi: 라이다가 180° 회전 마운트되어 실측 보정 (2026-05-22) -->
   <xacro:property name="laser_pose">
-    <origin xyz="0.13 0.0 0.420" rpy="0 0 0"/>
+    <origin xyz="0.13 0.0 0.420" rpy="0 0 ${pi}"/>
   </xacro:property>
   <!-- CAD 실측: camera_module [40] STEP(51,-8,358)mm -->

Commit message: fix(urdf): laser frame roll=pi (라이다 좌표계 좌우 미러링 보정)
yaw=pi(앞뒤 회전)는 좌우 반전을 야기하여 부적합. 라이다 데이터가
ROS 표준과 y축 미러링 관계인 것으로 확인됨. roll=pi로 frame 변환.

Co-Authored-By: Claude Opus 4.7 (1M context) <noreply@anthropic.com>

File: linorobot2_description/urdf/2wd_properties.urdf.xacro (robot description, xacro)
@@ -28,7 +28,8 @@
   <xacro:property name="wheel_mesh_file" value="" />
   <!-- CAD 실측: RPLIDAR [87] 상단(스캔면) STEP Z=417mm
-       rpy yaw=pi: 라이다가 180° 회전 마운트되어 실측 보정 (2026-05-22) -->
+       rpy roll=pi: 라이다 데이터 좌표계가 ROS 표준과 좌우 미러링 관계
+       (라이다 펌웨어 회전 방향 차이, 2026-05-22 실측 보정) -->
   <xacro:property name="laser_pose">
-    <origin xyz="0.13 0.0 0.420" rpy="0 0 ${pi}"/>
+    <origin xyz="0.13 0.0 0.420" rpy="${pi} 0 0"/>
   </xacro:property>
   <!-- CAD 실측: camera_module [40] STEP(51,-8,358)mm -->

Commit message: fix(urdf): laser frame rpy 원위치 (좌우 미러링은 scan_mask에서 처리)
URDF 회전(SO(3))으로는 미러링 표현 불가. scan_mask_node의
mirror_angle 옵션으로 데이터 레벨 처리.

Co-Authored-By: Claude Opus 4.7 (1M context) <noreply@anthropic.com>

File: linorobot2_description/urdf/2wd_properties.urdf.xacro (robot description, xacro)
@@ -27,9 +27,8 @@
   <xacro:property name="rear_caster_wheel" value="false" />
   <xacro:property name="wheel_mesh_file" value="" />
-  <!-- CAD 실측: RPLIDAR [87] 상단(스캔면) STEP Z=417mm
-       rpy roll=pi: 라이다 데이터 좌표계가 ROS 표준과 좌우 미러링 관계
-       (라이다 펌웨어 회전 방향 차이, 2026-05-22 실측 보정) -->
+  <!-- CAD 실측: RPLIDAR [87] 상단(스캔면) STEP Z=417mm.
+       라이다 좌우 미러링은 scan_mask_node의 mirror_angle 옵션으로 처리. -->
   <xacro:property name="laser_pose">
-    <origin xyz="0.13 0.0 0.420" rpy="${pi} 0 0"/>
+    <origin xyz="0.13 0.0 0.420" rpy="0 0 0"/>
   </xacro:property>
   <!-- CAD 실측: camera_module [40] STEP(51,-8,358)mm -->

Commit message: fix(urdf): laser frame yaw=pi (라이다 데이터 점대칭 상태 보정)
각 시도 결과를 종합 분석한 결과 라이다 데이터의 원본 상태가
점대칭(yaw=pi)인 것으로 확인. URDF yaw=pi로 frame 회전하면 identity.

Co-Authored-By: Claude Opus 4.7 (1M context) <noreply@anthropic.com>

File: linorobot2_description/urdf/2wd_properties.urdf.xacro (robot description, xacro)
@@ -28,7 +28,7 @@
   <xacro:property name="wheel_mesh_file" value="" />
   <!-- CAD 실측: RPLIDAR [87] 상단(스캔면) STEP Z=417mm.
-       라이다 좌우 미러링은 scan_mask_node의 mirror_angle 옵션으로 처리. -->
+       yaw=pi: 라이다 데이터가 점대칭 상태이므로 frame yaw=pi로 보정 (2026-05-22 실측). -->
   <xacro:property name="laser_pose">
-    <origin xyz="0.13 0.0 0.420" rpy="0 0 0"/>
+    <origin xyz="0.13 0.0 0.420" rpy="0 0 ${pi}"/>
   </xacro:property>
   <!-- CAD 실측: camera_module [40] STEP(51,-8,358)mm -->

Commit message: feat(description): rescuepang_v3.1 CAD 반영 + 카메라 리니어 액추에이터
신규 CAD(rescuepang_v3.1.stl)를 시뮬에 반영하고, 기존 구 CAD 기준
치수/센서 위치를 실측값으로 교체.

- 외형 메시: aed_robot.stl -> rescuepang_v3.1.stl
  (메시 +X=전방이라 회전 불필요, base_link가 메시 (-510,190,0)에 오도록 오프셋)
- 트랙폭 294 -> 370mm (인휠 중심 Y=±185). wheel_pos_y*2가 Gazebo
  wheel_separation으로 직결되어 시각/운동학 동시 반영
- 충돌박스 470x400 -> 720x487mm, 중심 X 0.160 -> 0.290 (섀시 X[-69.5,650])
- 캐스터 X 0.291 -> 0.595 (CAD 접지점). 충돌박스 중심 이동으로 무게중심이
  구 캐스터와 겹쳐 구동바퀴 하중이 0.3%가 되던 문제 해결 (-> 51%)
- 라이다 (0.13,0,0.420) -> (0.055,0,0.701) (원통 직경 76mm 중심/상단 실측)
- 뎁스카메라 (0.293,0,0.361) -> (0.562,-0.0035,0.597)
  L515 원반 실측(직경 59.4 x 두께 26.0mm), 틸트 없음. 값은 수납 위치
- camera_to_base_link: fixed -> prismatic (stroke 150mm, +X 전개)
  depth_sensor 매크로에 stroke 파라미터 추가(기본 0=fixed)하여 다른
  로봇 설정은 기존 동작 유지. Gazebo joint_pose_trajectory/joint_state_publisher
  플러그인으로 ros2_control 없이 구동

검증(Gazebo): 전진 1.115m(명령 1.0) / 회전 166도(명령 172도) /
라이다 측벽 1.950·1.951m 대칭, 자기몸체 오검출 0 / 붐 전개 0.1474, 수납 0.0004

주의: 라이다가 지면 0.861m로 올라가 0.86m 이하 장애물은 라이다 사각.
근거리 저장애물은 뎁스카메라(지면 0.757m, 1.45m 밖부터 바닥 커버)가 담당.

Co-Authored-By: Claude Opus 5 <noreply@anthropic.com>

File: linorobot2_description/urdf/2wd_properties.urdf.xacro (robot description, xacro)
@@ -4,13 +4,19 @@
        Visual STL은 전체 형상 유지하지만, 충돌 박스가 라이다 위치를 포함하면
        Gazebo lidar ray가 박스 내벽을 hit하여 phantom obstacle 발생 → 박스 상단을 라이다 아래로 -->
-  <xacro:property name="base_length" value="0.470" />
-  <xacro:property name="base_width" value="0.400" />
+  <!-- rescuepang_v3.1 CAD 실측: 섀시 X[-69.5,650] Y[±243.5] (전방 돌출부 X650~831은 주행 중 수납이라 제외) -->
+  <xacro:property name="base_length" value="0.720" />
+  <xacro:property name="base_width" value="0.487" />
   <xacro:property name="base_height" value="0.490" />
-  <!-- Z 범위: -0.102 ~ 0.388 (라이다 0.420 아래 3.2cm 마진) -->
-  <xacro:property name="base_origin_x" value="0.160" />
+  <!-- Z 범위: -0.102 ~ 0.388 (라이다 0.420 아래 3.2cm 마진) — 높이/Z중심은 기존 유지 -->
+  <xacro:property name="base_origin_x" value="0.290" />
   <xacro:property name="base_origin_y" value="0.000" />
   <xacro:property name="base_origin_z" value="0.143" />
   <xacro:property name="base_mass" value="13" />
-  <xacro:property name="base_mesh_file" value="package://linorobot2_description/meshes/aed_robot.stl" />
+  <!-- rescuepang_v3.1.stl: 메시 +X=전방이라 회전 불필요. base_link가 메시 (-510,190,0)에 오도록 오프셋.
+       (메시 실측: 인휠 직경 139mm→중심 X=-510, 좌우바퀴 Y=5/375→중심선 190, 메시 Z=0이 base_link 높이)
+       v3→v3.1은 뎁스카메라(L515)만 추가, 바퀴·라이다 기준점 및 외곽 치수 완전 동일 → 아래 값 그대로 유효 -->
+  <xacro:property name="base_mesh_file" value="package://linorobot2_description/meshes/rescuepang_v3.1.stl" />
+  <xacro:property name="base_mesh_xyz" value="0.510 -0.190 0.000" />
+  <xacro:property name="base_mesh_rpy" value="0 0 0" />
   <!-- CAD 실측: 인휠 직경 139mm → 반지름 69.5mm -->
   <xacro:property name="wheel_radius" value="0.0695" />
@@ -18,6 +24,7 @@
   <!-- base_link = 회전중심 (양 바퀴 축 중점). 바퀴는 base_link 원점에 위치 -->
   <xacro:property name="wheel_pos_x" value="0.0" />
-  <!-- 실측: 트랙폭 294mm / 2 = 147mm (CAD 340mm → 실측 보정) -->
-  <xacro:property name="wheel_pos_y" value="0.147" />
+  <!-- rescuepang_v3.1 CAD 실측: 트랙폭 370mm / 2 = 185mm (좌우 인휠 중심 Y=5/375).
+       ※ 실물(odrive_params.yaml track_width=0.294)은 구 조립체 실측값이라 v3 조립 후 재측정 필요. -->
+  <xacro:property name="wheel_pos_y" value="0.185" />
   <!-- 바퀴 중심: base_link 기준 z=-0.09m (인휠모터 축 높이, 본체 밑판 57.5mm 위에 본체가 있도록) -->
   <xacro:property name="wheel_pos_z" value="-0.09" />
@@ -27,16 +34,22 @@
   <xacro:property name="rear_caster_wheel" value="false" />
   <xacro:property name="wheel_mesh_file" value="" />
-  <!-- CAD 실측: RPLIDAR [87] 상단(스캔면) STEP Z=417mm.
-       yaw=pi: 라이다 데이터가 점대칭 상태이므로 frame yaw=pi로 보정 (2026-05-22 실측). -->
+  <!-- rescuepang_v3.1 CAD 실측: RPLIDAR 원통(직경 76mm) 중심 X=55mm, Y=0, 상단(스캔면) Z=701.3mm.
+       100x100 마운트 플레이트(Z 660) 위에 안착, 로봇 최상단. 구 CAD 대비 X -75mm / Z +281mm.
+       yaw=pi: 라이다 데이터가 점대칭 상태이므로 frame yaw=pi로 보정 (2026-05-22 실물 실측값 유지 — v3 조립 후 재확인 필요). -->
   <xacro:property name="laser_pose">
-    <origin xyz="0.13 0.0 0.420" rpy="0 0 ${pi}"/>
+    <origin xyz="0.055 0.0 0.701" rpy="0 0 ${pi}"/>
   </xacro:property>
-  <!-- CAD 실측: camera_module [40] STEP(51,-8,358)mm -->
+  <!-- rescuepang_v3.1 CAD 실측: RealSense L515 원반(직경 59.4mm·두께 26.0mm = L515 규격 61x26 일치).
+       렌즈면 X=561.8mm, 중심 Y=-3.5mm, Z=597.3mm. 틸트 없음(모든 Z단면 두께 26.0 균일) → 정면 수평.
+       지면 기준 높이 0.757m. 구 CAD 대비 X +269mm / Z +236mm. -->
   <xacro:property name="depth_sensor_pose">
-    <origin xyz="0.293 0.0 0.361" rpy="0 0 0"/>
+    <origin xyz="0.562 -0.0035 0.597" rpy="0 0 0"/>
   </xacro:property>
-  <!-- 시뮬용 RGB 카메라: depth_sensor와 동일 위치 (L515 마운트) -->
+  <!-- 카메라 리니어 액추에이터 스트로크 150mm (실물 사양, 2026-08-01 확인).
+       위 depth_sensor_pose = 수납 위치(주행 중). 전개 시 X = 0.562 + 0.150 = 0.712 -->
+  <xacro:property name="camera_boom_stroke" value="0.15" />
+  <!-- 시뮬용 RGB 카메라: depth_sensor와 동일 위치 (L515 마운트). 리니어 액추에이터에는 미연동(수납 위치 고정) -->
   <xacro:property name="rear_camera_sensor_pose">
-    <origin xyz="0.293 0.0 0.361" rpy="0 0 0"/>
+    <origin xyz="0.562 -0.0035 0.597" rpy="0 0 0"/>
   </xacro:property>
 </robot>

File: linorobot2_description/urdf/mech/base.urdf.xacro (robot description, xacro)
@@ -5,5 +5,5 @@
     <link name="base_link">
       <visual>
-        <origin xyz="0.285 -0.050 0.003" rpy="0 0 1.5708"/>
+        <origin xyz="${base_mesh_xyz}" rpy="${base_mesh_rpy}"/>
         <geometry>
           <mesh filename="${base_mesh_file}" scale="0.001 0.001 0.001"/>

File: linorobot2_description/urdf/robots/2wd.urdf.xacro (robot description, xacro)
@@ -40,9 +40,11 @@
     mass="${wheel_mass}"
   />
+  <!-- caster_x: rescuepang_v3 CAD 실측 접지점 X=595mm (좌우 Y=±191, 단일 중앙 캐스터로 근사).
+       구 0.291은 새 무게중심(base_origin_x=0.290)과 겹쳐 구동바퀴 하중이 0%가 됨 -->
   <xacro:if value="${front_caster_wheel}">
     <xacro:caster_wheel
       side="front"
       mass="0.01"
-      caster_x="0.291"
+      caster_x="0.595"
       caster_radius="0.060"
       wheel_radius="${wheel_radius}"
@@ -65,5 +67,7 @@
     <xacro:insert_block name="laser_pose" />
   </xacro:generic_laser>
-  <xacro:depth_sensor>
+  <!-- 카메라 리니어 액추에이터 스트로크 150mm (실물 사양).
+       depth_sensor_pose는 수납 위치이며, 전개 시 +X로 최대 0.15m 이동 -->
+  <xacro:depth_sensor stroke="${camera_boom_stroke}">
     <xacro:insert_block name="depth_sensor_pose" />
   </xacro:depth_sensor>

File: linorobot2_description/urdf/sensors/depth_sensor.urdf.xacro (robot description, xacro)
@@ -1,4 +1,7 @@
 <robot xmlns:xacro="http://ros.org/wiki/xacro">
-  <xacro:macro name="depth_sensor" params="*origin">
+  <!-- stroke: 리니어 액추에이터 스트로크(m). 0이면 고정 조인트(기존 동작 유지).
+       >0이면 camera_to_base_link가 prismatic이 되어 카메라를 +X로 전개할 수 있음.
+       origin은 항상 '수납(전개량 0)' 위치를 가리킨다. -->
+  <xacro:macro name="depth_sensor" params="*origin stroke:=0">
     <!-- Intel RealSense L515 -->
     <link name="camera_link">
@@ -24,9 +27,22 @@
       </inertial>
     </link>
-    <joint name="camera_to_base_link" type="fixed">
-      <parent link="base_link"/>
-      <child link="camera_link"/>
-      <xacro:insert_block name="origin"/>
-    </joint>
+    <xacro:if value="${stroke == 0}">
+      <joint name="camera_to_base_link" type="fixed">
+        <parent link="base_link"/>
+        <child link="camera_link"/>
+        <xacro:insert_block name="origin"/>
+      </joint>
+    </xacro:if>
+    <xacro:unless value="${stroke == 0}">
+      <!-- 리니어 액추에이터: 0=수납(주행), stroke=최대 전개 -->
+      <joint name="camera_to_base_link" type="prismatic">
+        <parent link="base_link"/>
+        <child link="camera_link"/>
+        <xacro:insert_block name="origin"/>
+        <axis xyz="1 0 0"/>
+        <limit lower="0" upper="${stroke}" effort="50" velocity="0.05"/>
+        <dynamics damping="20.0" friction="5.0"/>
+      </joint>
+    </xacro:unless>
     <link name="camera_depth_link"/>
     <joint name="camera_depth_joint" type="fixed">
@@ -62,4 +78,22 @@
       </sensor>
     </gazebo>
+    <!-- 리니어 액추에이터 구동/상태 (ros2_control 없이 Gazebo 플러그인으로 처리).
+         전개: /set_joint_trajectory (trajectory_msgs/JointTrajectory) 발행
+               joint_names=['camera_to_base_link'], positions=[0~stroke]
+               ⚠️ header.frame_id 는 반드시 'base_footprint' (Gazebo에서 고정조인트가
+                  base_footprint로 병합되어 base_link 링크는 존재하지 않음)
+         상태: /joint_states 의 camera_to_base_link 가 현재 전개량(m)
+         검증(2026-08-01): 전개 0.15 명령 → 0.1474, 수납 0 명령 → 0.0004 -->
+    <xacro:unless value="${stroke == 0}">
+      <gazebo>
+        <plugin name="camera_boom_traj" filename="libgazebo_ros_joint_pose_trajectory.so">
+          <update_rate>50</update_rate>
+        </plugin>
+        <plugin name="camera_boom_state" filename="libgazebo_ros_joint_state_publisher.so">
+          <update_rate>20</update_rate>
+          <joint_name>camera_to_base_link</joint_name>
+        </plugin>
+      </gazebo>
+    </xacro:unless>
   </xacro:macro>
 </robot>
