Commit message: feat(description): 카메라 틸트 관절 추가 (camera_mount_link + camera_tilt_joint)
- depth_sensor 매크로에 tilt 파라미터 신설(기본 0 = 관절 없음, 기존 설정 무영향)
- 틸트 축 +Y, 0~90°: 0=정면(+X), 90=바닥(-Z)
- joint_state_publisher에 camera_tilt_joint 등록
- 매크로 기본값 회귀 검증용 test_depth_sensor_macro.xacro 추가

Co-Authored-By: Claude Fable 5 <noreply@anthropic.com>

File: linorobot2_description/urdf/2wd_properties.urdf.xacro (robot description, xacro)
@@ -49,4 +49,6 @@
        위 depth_sensor_pose = 수납 위치(주행 중). 전개 시 X = 0.562 + 0.150 = 0.712 -->
   <xacro:property name="camera_boom_stroke" value="0.15" />
+  <!-- 카메라 틸트 서보 최대각 90° (실물 사양). 0=정면 주행, 1.5708=바닥 주시 -->
+  <xacro:property name="camera_tilt_max" value="1.5708" />
   <!-- 시뮬용 RGB 카메라: depth_sensor와 동일 위치 (L515 마운트). 리니어 액추에이터에는 미연동(수납 위치 고정) -->
   <xacro:property name="rear_camera_sensor_pose">

File: linorobot2_description/urdf/robots/2wd.urdf.xacro (robot description, xacro)
@@ -69,5 +69,5 @@
   <!-- 카메라 리니어 액추에이터 스트로크 150mm (실물 사양).
        depth_sensor_pose는 수납 위치이며, 전개 시 +X로 최대 0.15m 이동 -->
-  <xacro:depth_sensor stroke="${camera_boom_stroke}">
+  <xacro:depth_sensor stroke="${camera_boom_stroke}" tilt="${camera_tilt_max}">
     <xacro:insert_block name="depth_sensor_pose" />
   </xacro:depth_sensor>

File: linorobot2_description/urdf/sensors/depth_sensor.urdf.xacro (robot description, xacro)
@@ -2,6 +2,8 @@
   <!-- stroke: 리니어 액추에이터 스트로크(m). 0이면 고정 조인트(기존 동작 유지).
        >0이면 camera_to_base_link가 prismatic이 되어 카메라를 +X로 전개할 수 있음.
-       origin은 항상 '수납(전개량 0)' 위치를 가리킨다. -->
-  <xacro:macro name="depth_sensor" params="*origin stroke:=0">
+       origin은 항상 '수납(전개량 0)' 위치를 가리킨다.
+       tilt: 틸트 관절 최대각(rad). 0이면 관절 없이 카메라가 붐에 직결(기존 동작).
+             >0이면 camera_tilt_joint(+Y 회전)가 생겨 0=정면, tilt=바닥. -->
+  <xacro:macro name="depth_sensor" params="*origin stroke:=0 tilt:=0">
     <!-- Intel RealSense L515 -->
     <link name="camera_link">
@@ -30,5 +32,5 @@
       <joint name="camera_to_base_link" type="fixed">
         <parent link="base_link"/>
-        <child link="camera_link"/>
+        <child link="camera_mount_link"/>
         <xacro:insert_block name="origin"/>
       </joint>
@@ -38,9 +40,37 @@
       <joint name="camera_to_base_link" type="prismatic">
         <parent link="base_link"/>
-        <child link="camera_link"/>
+        <child link="camera_mount_link"/>
         <xacro:insert_block name="origin"/>
         <axis xyz="1 0 0"/>
         <limit lower="0" upper="${stroke}" effort="50" velocity="0.05"/>
         <dynamics damping="20.0" friction="5.0"/>
+      </joint>
+    </xacro:unless>
+    <!-- 붐 끝(리니어 액추에이터의 이동단). 틸트 서보가 여기 붙는다. -->
+    <link name="camera_mount_link">
+      <inertial>
+        <origin xyz="0 0 0" rpy="0 0 0"/>
+        <mass value="0.01"/>
+        <inertia ixx="0.000001" ixy="0.0" ixz="0.0"
+                 iyy="0.000001" iyz="0.0"
+                 izz="0.000001"/>
+      </inertial>
+    </link>
+    <xacro:if value="${tilt == 0}">
+      <joint name="camera_tilt_joint" type="fixed">
+        <parent link="camera_mount_link"/>
+        <child link="camera_link"/>
+        <origin xyz="0 0 0" rpy="0 0 0"/>
+      </joint>
+    </xacro:if>
+    <xacro:unless value="${tilt == 0}">
+      <!-- 틸트 서보: 0=정면(+X), tilt=바닥(-Z). +Y 회전이 +X를 -Z로 보낸다. -->
+      <joint name="camera_tilt_joint" type="revolute">
+        <parent link="camera_mount_link"/>
+        <child link="camera_link"/>
+        <origin xyz="0 0 0" rpy="0 0 0"/>
+        <axis xyz="0 1 0"/>
+        <limit lower="0" upper="${tilt}" effort="20" velocity="1.0"/>
+        <dynamics damping="2.0" friction="0.5"/>
       </joint>
     </xacro:unless>
@@ -93,4 +123,5 @@
           <update_rate>20</update_rate>
           <joint_name>camera_to_base_link</joint_name>
+          <joint_name>camera_tilt_joint</joint_name>
         </plugin>
       </gazebo>

Commit message: feat(urdf): 2wd에 SCARA 매크로 마운트
STL 실측 기준 (0.410, -0.099, -0.050), yaw 0.
4wd/mecanum/turtlebot/vattenkar는 호출하지 않아 영향 없음.

Co-Authored-By: Claude Fable 5 <noreply@anthropic.com>

File: linorobot2_description/urdf/2wd_properties.urdf.xacro (robot description, xacro)
@@ -55,3 +55,9 @@
     <origin xyz="0.562 -0.0035 0.597" rpy="0 0 0"/>
   </xacro:property>
+  <!-- SCARA(CPR 모듈) 마운트 — rescuepang_v3.1.stl 정점 실측 기준.
+       STL의 J1 축 (0.410, -0.099), 팔 회전면 Z 0.281.
+       URDF는 J1이 베이스 +0.33에 있으므로 z = 0.281 - 0.33 = -0.050.
+       STL에서 팔이 +X로 뻗어 있고 URDF 영점 자세도 로컬 +X라 yaw는 0. -->
+  <xacro:property name="scara_mount_xyz" value="0.410 -0.099 -0.050" />
+  <xacro:property name="scara_mount_rpy" value="0 0 0" />
 </robot>

File: linorobot2_description/urdf/robots/2wd.urdf.xacro (robot description, xacro)
@@ -10,4 +10,5 @@
   <xacro:include filename="$(find linorobot2_description)/urdf/sensors/depth_sensor.urdf.xacro" />
   <xacro:include filename="$(find linorobot2_description)/urdf/sensors/camera.urdf.xacro" />
+  <xacro:include filename="$(find scara_description)/urdf/scara_macro.xacro" />
   <xacro:include filename="$(find linorobot2_description)/urdf/controllers/diff_drive.urdf.xacro" />
   <xacro:base
@@ -78,4 +79,8 @@
     <xacro:insert_block name="rear_camera_sensor_pose" />
   </xacro:rgb_camera>
+  <!-- SCARA(CPR 모듈). 팔 회전면이 차체와 같은 높이이므로 타깃은 차체 앞(로버 X>0.65)에만 둔다. -->
+  <xacro:scara parent="base_link">
+    <origin xyz="${scara_mount_xyz}" rpy="${scara_mount_rpy}"/>
+  </xacro:scara>
   <xacro:diff_drive_controller
     wheel_separation="${wheel_pos_y * 2}"

Commit message: feat(mesh): SCARA 형상을 제거한 rescuepang_v3.1_no_scara.stl
원본 메시에는 SCARA가 형상으로 들어 있는데 base_link에 붙은 통짜 STL이라
움직이지 않는다. URDF 관절(scara_base_link~crank_link)이 기본도형으로 팔을
렌더하므로 화면에 팔이 두 개로 보였다.

- 제거: 팔 본체(X 0.354~0.835, Y -0.190~-0.019, Z 0~0.400)
        + 크랭크 밑면(X 0.680~0.835, 같은 Y, Z -0.020~0)   총 59,327 삼각형
- 330,912 → 271,585 삼각형 (16.5MB → 13.6MB)
- 로버 X 최댓값 0.831 → 0.640 (차체 앞끝과 일치)
- X 0.36~0.54 / Z -0.03~0 구간은 섀시 바닥과 구분이 안 돼 의도적으로 남김
- 원본은 CAD 실측 참조용으로 보존

검증: 3면 투영으로 제거분이 J1→J2→크랭크 체인임을, 남은 쪽에 섀시·바퀴·
라이다·카메라 마운트가 온전함을 확인. Gazebo 재기동 후 메시 오류 0,
컨트롤러 3개 active, SCARA 4관절 정상.

Co-Authored-By: Claude Fable 5 <noreply@anthropic.com>

File: linorobot2_description/urdf/2wd_properties.urdf.xacro (robot description, xacro)
@@ -16,5 +16,9 @@
        (메시 실측: 인휠 직경 139mm→중심 X=-510, 좌우바퀴 Y=5/375→중심선 190, 메시 Z=0이 base_link 높이)
        v3→v3.1은 뎁스카메라(L515)만 추가, 바퀴·라이다 기준점 및 외곽 치수 완전 동일 → 아래 값 그대로 유효 -->
-  <xacro:property name="base_mesh_file" value="package://linorobot2_description/meshes/rescuepang_v3.1.stl" />
+  <!-- SCARA 형상을 제거한 메시를 쓴다. 원본(rescuepang_v3.1.stl)에는 팔이 형상으로
+       들어 있는데 그건 base_link에 붙은 통짜 메시라 움직이지 않는다. 움직이는 URDF
+       관절(scara_base_link~crank_link)과 겹쳐 보여 화면에 팔이 둘로 보였다.
+       원본은 CAD 실측 참조용으로 같은 폴더에 보존. -->
+  <xacro:property name="base_mesh_file" value="package://linorobot2_description/meshes/rescuepang_v3.1_no_scara.stl" />
   <xacro:property name="base_mesh_xyz" value="0.510 -0.190 0.000" />
   <xacro:property name="base_mesh_rpy" value="0 0 0" />

Commit message: fix(urdf): 무게중심을 충돌박스에서 분리 + 캐스터 높이 연동 + 바퀴 토크 전달
세 가지 모두 "파라미터를 받아놓고 쓰지 않던" 같은 유형의 누락이다.

1. base 매크로가 <collision>과 <inertial>에 같은 origin을 써서, 충돌박스를
   CAD 실측(중심 x=0.290)에 맞추자 무게중심까지 같이 앞으로 끌려갔다. 실제
   질량은 인휠모터(바퀴축)와 배터리·ODrive가 있는 뒤쪽에 몰려 있다.
   com_offset_x(기본 0, 다른 로봇 설정은 동작 불변)로 분리해 x=0.150 적용.
   구동륜 하중 51% -> 75%.

2. caster_wheel 매크로가 wheel_radius/wheel_pos_z를 받으면서 z를 -0.100으로
   하드코딩하고 있었다. 인휠모터 실측 반영(wheel_radius 0.045->0.0695,
   wheel_pos_z -0.03->-0.09) 때 함께 갱신되지 않아 캐스터가 구동륜보다
   0.5mm 아래로 내려가 있었다. 업스트림 방식대로 수식으로 복원.
   바퀴/캐스터 최하점 모두 z=-0.1595로 일치 (SDF 덤프 검증).

3. diff_drive 매크로가 wheel_torque를 받으면서 플러그인에 넘기지 않아
   gazebo_ros_diff_drive 기본값 5.0 N·m으로 돌고 있었다. max_wheel_torque로
   전달. 아울러 max_wheel_acceleration 1.0은 바퀴 기준이라 로봇 선가속
   0.0695 m/s²에 불과해 0.8 m/s 도달에 11.5초가 걸렸다 -> 15.0.
   직진이 0.5초 내 100% 도달로 개선.

Co-Authored-By: Claude Fable 5 <noreply@anthropic.com>

File: linorobot2_description/urdf/2wd_properties.urdf.xacro (robot description, xacro)
@@ -13,4 +13,10 @@
   <xacro:property name="base_origin_z" value="0.143" />
   <xacro:property name="base_mass" value="13" />
+  <!-- 무게중심 보정: 충돌박스 중심(base_origin_x=0.290)은 CAD 외곽 기준이라 실제 질량 분포와
+       다르다. 인휠모터는 바퀴축(x=0), 배터리·ODrive는 뒤~중앙에 있고 앞쪽 X 0.4~0.65는
+       SCARA 마운트와 빈 공간이다. 무게중심을 0.290 → 0.150으로 당겨 구동바퀴 하중을
+       51% → 75%로 회복시킨다 (캐스터 x=0.595 기준).
+       ※ 0.150은 추정치다. 실물 무게중심 실측 시 그 값으로 교체할 것. -->
+  <xacro:property name="base_com_offset_x" value="-0.140" />
   <!-- rescuepang_v3.1.stl: 메시 +X=전방이라 회전 불필요. base_link가 메시 (-510,190,0)에 오도록 오프셋.
        (메시 실측: 인휠 직경 139mm→중심 X=-510, 좌우바퀴 Y=5/375→중심선 190, 메시 Z=0이 base_link 높이)

File: linorobot2_description/urdf/controllers/diff_drive.urdf.xacro (robot description, xacro)
@@ -12,5 +12,12 @@
         <wheel_separation>${wheel_separation}</wheel_separation>
         <wheel_diameter>${wheel_radius * 2}</wheel_diameter>
-        <max_wheel_acceleration>1.0</max_wheel_acceleration>
+        <!-- 이 값은 바퀴 각가속(rad/s²) 기준이라 로봇 선가속으로 환산하면
+             1.0 x wheel_radius = 0.0695 m/s² 밖에 안 된다. 0.8 m/s 도달에 11.5초가
+             걸려 주행 내내 가속 구간에 머물렀다. velocity_smoother의 max_accel
+             1.0 m/s²를 실제로 내려면 바퀴 기준 1.0/0.0695 = 14.4 rad/s²가 필요하다. -->
+        <max_wheel_acceleration>15.0</max_wheel_acceleration>
+        <!-- 매크로가 wheel_torque를 받으면서 플러그인에 넘기지 않아
+             gazebo_ros_diff_drive 기본값 5.0 N·m으로 돌고 있었다. -->
+        <max_wheel_torque>${wheel_torque}</max_wheel_torque>
         <robot_base_frame>base_footprint</robot_base_frame>
         <publish_odom>true</publish_odom>

File: linorobot2_description/urdf/mech/base.urdf.xacro (robot description, xacro)
@@ -1,5 +1,5 @@
 <?xml version="1.0"?>
 <robot xmlns:xacro="http://ros.org/wiki/xacro">
-  <xacro:macro name="base" params="length width height mass wheel_radius wheel_pos_z origin_x origin_y origin_z">
+  <xacro:macro name="base" params="length width height mass wheel_radius wheel_pos_z origin_x origin_y origin_z com_offset_x:=0">
     <link name="base_footprint"/>
     <link name="base_link">
@@ -28,6 +28,10 @@
         </geometry>
       </collision>
+      <!-- 무게중심은 충돌박스 기하중심과 다르다. 충돌박스는 CAD 외곽이지만 실제 질량은
+           인휠모터(바퀴축)와 배터리·ODrive가 있는 뒤쪽에 몰려 있다. 둘을 같은 origin으로
+           묶으면 무게중심이 앞으로 끌려가 구동바퀴 하중이 빠지고 회전·가속이 죽는다.
+           com_offset_x 기본 0이라 다른 로봇 설정은 기존 동작 그대로다. -->
       <inertial>
-        <origin xyz="${origin_x} ${origin_y} ${origin_z}" rpy="0 0 0"/>
+        <origin xyz="${origin_x + com_offset_x} ${origin_y} ${origin_z}" rpy="0 0 0"/>
         <mass value="${mass}"/>
         <inertia ixx="${(1/12) * mass * ((width  * width)  + (height * height))}" ixy="0.0" ixz="0.0"

File: linorobot2_description/urdf/mech/caster_wheel.urdf.xacro (robot description, xacro)
@@ -35,5 +35,11 @@
       <parent link="base_link"/>
       <child link="${side}_caster_wheel_link"/>
-      <origin xyz="${caster_wheel_x} 0 -0.100" rpy="0 0 0"/>
+      <!-- 캐스터 최하점을 구동바퀴 최하점에 맞춘다.
+           z를 -0.100으로 하드코딩하던 값은 인휠모터 실측(wheel_radius 0.045→0.0695,
+           wheel_pos_z -0.03→-0.09) 반영 시 함께 갱신되지 않아, 캐스터가 바퀴보다
+           0.5mm 아래로 내려가 있었다. 그 결과 로봇이 캐스터에 얹혀 구동바퀴 접지가
+           빠지면서 회전과 가속이 제대로 안 됐다.
+           매크로가 wheel_radius/wheel_pos_z를 이미 받고 있으므로 그걸로 계산한다. -->
+      <origin xyz="${caster_wheel_x} 0 ${wheel_pos_z - wheel_radius + caster_wheel_radius}" rpy="0 0 0"/>
     </joint>
   </xacro:macro>

File: linorobot2_description/urdf/robots/2wd.urdf.xacro (robot description, xacro)
@@ -26,4 +26,5 @@
     origin_y="${base_origin_y}"
     origin_z="${base_origin_z}"
+    com_offset_x="${base_com_offset_x}"
 />
   <xacro:wheel

Commit message: fix(urdf): 로봇 형상 실측값 반영 — 트랙폭 0.325, IMU·라이다 위치
v3.1 조립체를 실측해 CAD 추정값과 linorobot2 기본값을 대체한다.

- track_width: wheel_pos_y 0.185 → 0.1625 (실측 325mm)
  CAD 370mm 도 구 조립체 294mm 도 아니었다. 실물이 0.294 로 돌고 있어
  제자리 회전 오도메트리가 약 11% 과대 보고되고 있었다(90도마다 10도 오차).
- 라이다 Z: 0.701 → 0.7705 (지면~스캔면 930mm, base_link 는 지면+0.1595)
- IMU: (-0.0075, 0, 0.0135) → (-0.03, 0, 0.0155)
  구값은 linorobot2 원본 기본값이었고 이 로봇을 측정한 적이 없었다.
  EKF 는 IMU 에서 z축 각속도만 융합하므로 영향은 제한적이나 값을 맞춰둔다.

Co-Authored-By: Claude Opus 5 <noreply@anthropic.com>

File: linorobot2_description/urdf/2wd_properties.urdf.xacro (robot description, xacro)
@@ -43,7 +43,8 @@
   <!-- base_link = 회전중심 (양 바퀴 축 중점). 바퀴는 base_link 원점에 위치 -->
   <xacro:property name="wheel_pos_x" value="0.0" />
-  <!-- rescuepang_v3.1 CAD 실측: 트랙폭 370mm / 2 = 185mm (좌우 인휠 중심 Y=5/375).
-       ※ 실물(odrive_params.yaml track_width=0.294)은 구 조립체 실측값이라 v3 조립 후 재측정 필요. -->
-  <xacro:property name="wheel_pos_y" value="0.185" />
+  <!-- 실물 실측 (2026-08-20): 좌우 인휠 중심 사이 325mm / 2 = 162.5mm.
+       CAD 값 370mm 및 구 조립체 실측값 294mm 를 모두 대체한다.
+       odrive_params.yaml 의 track_width 도 같은 값(0.325)이어야 회전 오도메트리가 맞는다. -->
+  <xacro:property name="wheel_pos_y" value="0.1625" />
   <!-- 바퀴 중심: base_link 기준 z=-0.09m (인휠모터 축 높이, 본체 밑판 57.5mm 위에 본체가 있도록) -->
   <xacro:property name="wheel_pos_z" value="-0.09" />
@@ -55,7 +56,9 @@
   <!-- rescuepang_v3.1 CAD 실측: RPLIDAR 원통(직경 76mm) 중심 X=55mm, Y=0, 상단(스캔면) Z=701.3mm.
        100x100 마운트 플레이트(Z 660) 위에 안착, 로봇 최상단. 구 CAD 대비 X -75mm / Z +281mm.
-       yaw=pi: 라이다 데이터가 점대칭 상태이므로 frame yaw=pi로 보정 (2026-05-22 실물 실측값 유지 — v3 조립 후 재확인 필요). -->
+       yaw=pi: 라이다 데이터가 점대칭 상태이므로 frame yaw=pi로 보정 (2026-05-22 실물 실측값 유지).
+       Z 는 실물 실측(2026-08-20): 지면~스캔면 930mm. base_link 는 지면보다 159.5mm 위
+       (wheel_radius 0.0695 + |wheel_pos_z| 0.09) 이므로 0.930 - 0.1595 = 0.7705. -->
   <xacro:property name="laser_pose">
-    <origin xyz="0.055 0.0 0.701" rpy="0 0 ${pi}"/>
+    <origin xyz="0.055 0.0 0.7705" rpy="0 0 ${pi}"/>
   </xacro:property>
   <!-- rescuepang_v3.1 CAD 실측: RealSense L515 원반(직경 59.4mm·두께 26.0mm = L515 규격 61x26 일치).

File: linorobot2_description/urdf/sensors/imu.urdf.xacro (robot description, xacro)
@@ -5,5 +5,7 @@
       <parent link="base_link"/>
       <child link="imu_link"/>
-      <origin xyz="-0.0075 0 0.0135" rpy="0 0 0"/>
+      <!-- 실물 실측 (2026-08-20): 바퀴축 중점 기준 뒤로 30mm, 좌우 중앙,
+           지면에서 175mm. base_link 가 지면보다 159.5mm 위이므로 z = 0.175 - 0.1595. -->
+      <origin xyz="-0.03 0 0.0155" rpy="0 0 0"/>
     </joint>
     <gazebo reference="imu_link">

Commit message: fix(urdf): 뎁스카메라 높이를 실측 865mm 로 (CAD 대비 +108mm)
지면~컬러 렌즈를 직접 재니 865mm 였다. CAD v3.1 값(Z=597.3mm, 지면 757mm)은
실물 조립과 108mm 차이가 난다. laser_pose 와 같은 방식으로 실측을 우선한다.
  z = 0.865 - 0.1595(base_link 지상고) = 0.7055

컬러/뎁스 구분은 이 모델에서 의미가 없다 — camera_depth_link 가 camera_link 에
대해 회전만 갖고 위치 오프셋이 0 이다. 실물 조리개 간격은 realsense2_camera 가
공장 extrinsic 으로 직접 TF 를 내며 1cm 이내다.

Co-Authored-By: Claude Opus 5 <noreply@anthropic.com>

File: linorobot2_description/urdf/2wd_properties.urdf.xacro (robot description, xacro)
@@ -63,8 +63,15 @@
   </xacro:property>
   <!-- rescuepang_v3.1 CAD 실측: RealSense L515 원반(직경 59.4mm·두께 26.0mm = L515 규격 61x26 일치).
-       렌즈면 X=561.8mm, 중심 Y=-3.5mm, Z=597.3mm. 틸트 없음(모든 Z단면 두께 26.0 균일) → 정면 수평.
-       지면 기준 높이 0.757m. 구 CAD 대비 X +269mm / Z +236mm. -->
+       렌즈면 X=561.8mm, 중심 Y=-3.5mm. 틸트 없음(모든 Z단면 두께 26.0 균일) → 정면 수평.
+       Z 는 실물 실측(2026-08-23): 지면~컬러 렌즈 865mm. base_link 는 지면보다 159.5mm 위
+       (wheel_radius 0.0695 + |wheel_pos_z| 0.09) 이므로 0.865 - 0.1595 = 0.7055.
+       CAD(v3.1) 값은 Z=597.3mm(지면 757mm)였는데 실물이 108mm 더 높게 조립됐다.
+       laser_pose 와 같은 방식으로 실측을 우선한다.
+       컬러/뎁스 구분: 아래 camera_depth_link 가 camera_link 에 대해 회전만 갖고
+       위치 오프셋이 0 이라, 이 모델에서 둘은 같은 점이다. 실물의 조리개 간격은
+       realsense2_camera 노드가 공장 extrinsic 으로 직접 TF 를 내며 1cm 이내라
+       줄자 오차보다 작다. -->
   <xacro:property name="depth_sensor_pose">
-    <origin xyz="0.562 -0.0035 0.597" rpy="0 0 0"/>
+    <origin xyz="0.562 -0.0035 0.7055" rpy="0 0 0"/>
   </xacro:property>
   <!-- 카메라 리니어 액추에이터 스트로크 150mm (실물 사양, 2026-08-01 확인).
