Commit message: Fix scara include failure and controller spawn error handling
- 2wd.urdf.xacro: add use_scara xacro arg (default true) so a missing
  scara_description install no longer crashes the whole real-robot
  bringup LaunchDescription (lidar/ODrive/IMU included).
- gazebo.launch.py: OnProcessExit handlers now check event.returncode
  and log a warning instead of silently chaining controller spawners
  after a failed spawn, which previously let ik_node's P-loop drive
  the arm open-loop into its joint limits.
- gazebo.launch.py: drop the now-unused Command import.

Co-Authored-By: Claude Fable 5 <noreply@anthropic.com>

File: linorobot2_description/urdf/robots/2wd.urdf.xacro (robot description, xacro)
@@ -1,4 +1,6 @@
 <?xml version="1.0"?>
 <robot name="linorobot2_2wd" xmlns:xacro="http://ros.org/wiki/xacro">
+  <xacro:arg name="use_scara" default="true"/>
+  <xacro:property name="use_scara" value="$(arg use_scara)"/>
   <xacro:include filename="$(find linorobot2_description)/urdf/2wd_properties.urdf.xacro" />
   <xacro:include filename="$(find linorobot2_description)/urdf/mech/base.urdf.xacro" />
@@ -10,5 +12,7 @@
   <xacro:include filename="$(find linorobot2_description)/urdf/sensors/depth_sensor.urdf.xacro" />
   <xacro:include filename="$(find linorobot2_description)/urdf/sensors/camera.urdf.xacro" />
-  <xacro:include filename="$(find scara_description)/urdf/scara_macro.xacro" />
+  <xacro:if value="${use_scara}">
+    <xacro:include filename="$(find scara_description)/urdf/scara_macro.xacro" />
+  </xacro:if>
   <xacro:include filename="$(find linorobot2_description)/urdf/controllers/diff_drive.urdf.xacro" />
   <xacro:base
@@ -80,7 +84,9 @@
   </xacro:rgb_camera>
   <!-- SCARA(CPR 모듈). 팔 회전면이 차체와 같은 높이이므로 타깃은 차체 앞(로버 X>0.65)에만 둔다. -->
-  <xacro:scara parent="base_link">
-    <origin xyz="${scara_mount_xyz}" rpy="${scara_mount_rpy}"/>
-  </xacro:scara>
+  <xacro:if value="${use_scara}">
+    <xacro:scara parent="base_link">
+      <origin xyz="${scara_mount_xyz}" rpy="${scara_mount_rpy}"/>
+    </xacro:scara>
+  </xacro:if>
   <xacro:diff_drive_controller
     wheel_separation="${wheel_pos_y * 2}"
