Commit message: fix: gazebo 블록 위치 + RPP 파라미터명 오타
둘 다 조용히 무시되던 것들이다.

- base.urdf.xacro: <gazebo reference="base_link">가 <link> 안에 있었다.
  URDF 파서가 무시해 Gazebo 머티리얼이 적용되지 않았다. 업스트림처럼
  <link> 바깥으로 옮겼다. 생성 SDF에서 ambient/diffuse/specular 적용 확인.

- navigation_sim.yaml: rotate_to_heading_min_theta는 humble RPP에 없는
  이름이다(실물 config는 rotate_to_heading_min_angle로 올바름). 조용히
  무시되어 기본값 0.785가 적용돼 왔다. 이름을 바로잡되 값은 그동안 실제로
  동작하던 0.785를 유지한다 — 원래 의도했던 0.1은 5.7°만 틀어져도 제자리
  회전을 걸어 과하다.

Co-Authored-By: Claude Fable 5 <noreply@anthropic.com>

File: linorobot2_description/urdf/mech/base.urdf.xacro (robot description, xacro)
@@ -13,13 +13,4 @@
         </material>
       </visual>
-    <gazebo reference="base_link">
-      <visual>
-        <material>
-          <ambient>0.3 0.3 0.3 1.0</ambient>
-          <diffuse>0.5 0.5 0.5 1.0</diffuse>
-          <specular>0.2 0.2 0.2 1.0</specular>
-        </material>
-      </visual>
-    </gazebo>
       <collision>
         <origin xyz="${origin_x} ${origin_y} ${origin_z}" rpy="0 0 0"/>
@@ -40,4 +31,15 @@
       </inertial>
     </link>
+    <!-- <gazebo>는 <link> 바깥에 와야 한다. 안에 두면 URDF 파서가 무시해
+         Gazebo 머티리얼이 적용되지 않는다 (업스트림도 바깥). -->
+    <gazebo reference="base_link">
+      <visual>
+        <material>
+          <ambient>0.3 0.3 0.3 1.0</ambient>
+          <diffuse>0.5 0.5 0.5 1.0</diffuse>
+          <specular>0.2 0.2 0.2 1.0</specular>
+        </material>
+      </visual>
+    </gazebo>
     <joint name="base_to_footprint" type="fixed">
       <parent link="base_footprint"/>
