Commit message: fix(description): camera_mount_link 관성값을 1e-6→2.5e-5로 상향 (NaN 관절 회귀 수정)
camera_to_base_link(prismatic) 위치가 시뮬 시작 직후부터 NaN이 되고
camera_tilt_joint(revolute)가 전혀 움직이지 않던 회귀(4a049c2)의 근본 원인:
camera_mount_link의 회전 관성(1e-6 kg·m²)이 camera_tilt_joint의 damping
계수(2.0)에 비해 물리 스텝(0.001s, aed_corridor.world)에서 ODE가 감당하기엔
너무 작아, 시뮬 시작 즉시 해당 관절 상태가 발산 → 두 조인트가 공유하는
camera_mount_link 강체 상태 전체가 오염되어 prismatic 쪽도 NaN으로 전파됨.

4개 A/B 실험으로 확인:
- mass=0.01/I=1e-6 (기존): NaN
- mass=0.1 /I=2.5e-5      : 정상
- mass=0.1 /I=1e-6        : NaN (mass만 올려선 불충분 — 관성이 핵심 변수)
- mass=0.01/I=2.5e-5      : 정상 (mass는 그대로, 관성만 올려도 충분)

mass는 원래 값(0.01) 유지, inertia만 camera_link와 동일한 2.5e-5로 상향.
링크 체인 구조·틸트 축/범위·tilt=0 기본 동작은 변경 없음.

Co-Authored-By: Claude Fable 5 <noreply@anthropic.com>

File: linorobot2_description/urdf/sensors/depth_sensor.urdf.xacro (robot description, xacro)
@@ -52,7 +52,7 @@
         <origin xyz="0 0 0" rpy="0 0 0"/>
         <mass value="0.01"/>
-        <inertia ixx="0.000001" ixy="0.0" ixz="0.0"
-                 iyy="0.000001" iyz="0.0"
-                 izz="0.000001"/>
+        <inertia ixx="0.000025" ixy="0.0" ixz="0.0"
+                 iyy="0.000025" iyz="0.0"
+                 izz="0.000025"/>
       </inertial>
     </link>

Commit message: fix(urdf): 카메라가 시뮬 화면에 보이도록 비주얼 교체
camera_link의 visual이 realsense2_description의 l515.dae를 절대경로로
참조했는데 그 패키지가 설치돼 있지 않아 아무것도 렌더되지 않았다.
그래서 붐 전개(150mm)와 틸트(90°)가 화면에서 안 보였다. 관절은 정상
동작 중이었다 — TF상 camera_link의 +X축이 바닥을 향하는 것으로 확인.

이미 있던 충돌 원통과 같은 치수(⌀61 x 26mm)의 기본 도형으로 바꿨다.
외부 패키지 의존이 없어 컨테이너를 다시 만들어도 깨지지 않는다.

섀시 STL에도 L515 원반이 형상으로 들어 있어(v3→v3.1 추가분) 수납 시
겹치므로 Gazebo/Blue를 줘 움직이는 쪽을 구분할 수 있게 했다.

깊이 센서 영향 없음 확인: 자기 형상에 가리지 않는다(최소 거리 1.440m,
near clip 0.25m). 유효화소 60.2%.

Co-Authored-By: Claude Opus 5 <noreply@anthropic.com>

File: linorobot2_description/urdf/sensors/depth_sensor.urdf.xacro (robot description, xacro)
@@ -8,8 +8,11 @@
     <!-- Intel RealSense L515 -->
     <link name="camera_link">
+      <!-- 충돌과 같은 원통. 원래 realsense2_description의 l515.dae를 참조했는데
+           그 패키지가 설치돼 있지 않아 아무것도 안 그려졌고, 그래서 붐 전개와
+           틸트가 화면에서 보이지 않았다(2026-08-08). 기본 도형이라 외부 의존이 없다. -->
       <visual>
-        <origin xyz="0 0 0" rpy="0 0 0"/>
+        <origin xyz="0 0 0" rpy="0 1.5708 0"/>
         <geometry>
-          <mesh filename="file:///opt/ros/humble/share/realsense2_description/meshes/l515.dae"/>
+          <cylinder radius="0.0305" length="0.026"/>
         </geometry>
       </visual>
@@ -83,4 +86,7 @@
     <!-- Gazebo Classic 11 depth camera — L515 스펙 -->
     <gazebo reference="camera_link">
+      <!-- 섀시 STL에도 L515 원반이 형상으로 들어 있어(v3→v3.1 추가분) 수납 시
+           겹친다. 색을 달리해야 어느 쪽이 움직이는 카메라인지 구분된다. -->
+      <material>Gazebo/Blue</material>
       <sensor name="camera" type="depth">
         <always_on>true</always_on>
